Commit message: add camera_link

File: kortex_description/robots/kortex_robot.xacro (robot description, xacro)
@@ -1,52 +1,60 @@
 <?xml version="1.0"?>
 <robot xmlns:xacro="http://ros.org/wiki/xacro">
-    <xacro:macro name="load_robot" params="arm gripper sim">
-        <!-- Arguments -->
-        <xacro:property name="arm" value="$(arg arm)" />
-        <xacro:property name="gripper" default="$(arg gripper)" />
-        <xacro:property name="sim" default="$(arg sim)" />
-        <!-- Files to include -->
-        <xacro:include filename="$(find kortex_description)/arms/$(arg arm)/urdf/$(arg arm)_macro.xacro" />
-        <xacro:unless value="${not gripper}">
-            <xacro:include filename="$(find kortex_description)/grippers/$(arg gripper)/urdf/$(arg gripper)_macro.xacro" />
-        </xacro:unless>
-        <xacro:if value="$(arg sim)">
-            <!-- Arm transmission elements-->
-            <xacro:include filename="$(find kortex_description)/arms/$(arg arm)/urdf/$(arg arm)_transmission_macro.xacro" />
-            <!-- Gripper transmission elements if there is a gripper-->
-            <xacro:unless value="${not gripper}">
-                <xacro:include filename="$(find kortex_description)/grippers/$(arg gripper)/urdf/$(arg gripper)_transmission_macro.xacro" />
-            </xacro:unless>
-        </xacro:if>
-        <!-- Run the macros -->
-        <!-- For gazebo-->
-        <xacro:if value="$(arg sim)">
-            <link name="world" />
-            <joint name="world_to_root" type="fixed">
-                <child link="base_link" />
-                <parent link="world" />
-                <origin xyz="0 0 0" rpy="0 0 0" />
-            </joint>
-        </xacro:if>
-        <!-- Load the arm -->
-        <xacro:load_arm parent="">
-            <origin xyz="0 0 0" rpy="0 0 0"/>
-        </xacro:load_arm>
-        <!-- Load the gripper -->
-        <xacro:unless value="${not gripper}">
-            <xacro:load_gripper parent="${last_arm_link}"/> <!-- last_arm_link is defined in "$(find kortex_description)/arms/$(arg arm)/urdf/$(arg arm)_macro.xacro" -->
-        </xacro:unless>
-        <!-- Load the Gazebo transmissions and gazebo_ros_control plugin -->
-        <xacro:if value="$(arg sim)">
-            <xacro:load_gazebo_arm_transmissions/>
-            <xacro:unless value="${not gripper}">
-                <xacro:load_gazebo_gripper_transmissions/>
-            </xacro:unless>
-            <gazebo>
-                <plugin name="gazebo_ros_control" filename="libgazebo_ros_control.so">
-                    <legacyModeNS>true</legacyModeNS>
-                </plugin>
-            </gazebo>
-        </xacro:if>
-    </xacro:macro>
+  <xacro:macro name="load_robot" params="arm gripper sim">
+    <!-- Arguments -->
+    <xacro:property name="arm" value="$(arg arm)" />
+    <xacro:property name="gripper" default="$(arg gripper)" />
+    <xacro:property name="sim" default="$(arg sim)" />
+    <!-- Files to include -->
+    <xacro:include filename="$(find kortex_description)/arms/$(arg arm)/urdf/$(arg arm)_macro.xacro" />
+    <xacro:unless value="${not gripper}">
+      <xacro:include filename="$(find kortex_description)/grippers/$(arg gripper)/urdf/$(arg gripper)_macro.xacro" />
+    </xacro:unless>
+    <xacro:if value="$(arg sim)">
+      <!-- Arm transmission elements-->
+      <xacro:include filename="$(find kortex_description)/arms/$(arg arm)/urdf/$(arg arm)_transmission_macro.xacro" />
+      <!-- Gripper transmission elements if there is a gripper-->
+      <xacro:unless value="${not gripper}">
+        <xacro:include filename="$(find kortex_description)/grippers/$(arg gripper)/urdf/$(arg gripper)_transmission_macro.xacro" />
+      </xacro:unless>
+    </xacro:if>
+    <!-- Run the macros -->
+    <!-- For gazebo-->
+    <xacro:if value="$(arg sim)">
+      <link name="world" />
+      <joint name="world_to_root" type="fixed">
+        <child link="base_link" />
+        <parent link="world" />
+        <origin xyz="0 0 0" rpy="0 0 0" />
+      </joint>
+    </xacro:if>
+    <!-- Load the arm -->
+    <xacro:load_arm parent="">
+      <origin xyz="0 0 0" rpy="0 0 0"/>
+    </xacro:load_arm>
+    <!-- Load the gripper -->
+    <xacro:unless value="${not gripper}">
+      <xacro:load_gripper parent="${last_arm_link}"/>
+      <!-- last_arm_link is defined in "$(find kortex_description)/arms/$(arg arm)/urdf/$(arg arm)_macro.xacro" -->
+    </xacro:unless>
+    <!-- Camera link -->
+    <link name="camera_link"/>
+    <joint name="camera_link_joint" type="fixed">
+      <origin xyz="0 0.05639 -0.00305" rpy="0 0 3.1415926" />
+      <parent link="end_effector_link" />
+      <child link="camera_link" />
+    </joint>
+    <!-- Load the Gazebo transmissions and gazebo_ros_control plugin -->
+    <xacro:if value="$(arg sim)">
+      <xacro:load_gazebo_arm_transmissions/>
+      <xacro:unless value="${not gripper}">
+        <xacro:load_gazebo_gripper_transmissions/>
+      </xacro:unless>
+      <gazebo>
+        <plugin name="gazebo_ros_control" filename="libgazebo_ros_control.so">
+          <legacyModeNS>true</legacyModeNS>
+        </plugin>
+      </gazebo>
+    </xacro:if>
+  </xacro:macro>
 </robot>
